File: pcb/keyboard-100x100-minif4-dual-rgb-reversible.kicad_pcb (KiCad board)
At the start: 2 copper layers, 100 x 100 mm, 110 parts, among them J1 TRRS, J2 TRRS, J3 Conn_01x04_Female, M1 Motor_DC, Q1 Q_NPN_BCE, U1 BluePill_or_MiniF4, U2 SN74LVC1T45DBV

Commit message: more tidying
Parts:
- turned D_BL_4 to 0 degrees
Routing:
- net /5V: track 993.1 -> 1001.9 mm
- net /DOUT_BL: track 23.2 -> 32.0 mm
- net /SW15: track 133.6 -> 140.7 mm, vias 16 -> 14
- net /GND: track 221.5 -> 214.7 mm, vias 34 -> 33
- net Net-(D_BL_3-Pad4): track 84.8 -> 86.9 mm, vias 12 -> 10
- net Net-(D_24-Pad2): track 39.9 -> 38.6 mm
- net /DOUT_2: vias 11 -> 9
