File: pcb/keyboard-x2-lumberjack-arm.kicad_pcb (KiCad board)
At the start: 2 copper layers, 285 x 94.2 mm, 144 parts, among them J1 USB_C_Receptacle_USB2.0, U1 BluePill_or_MiniF4_DIP40, U2 SN74LVC1T45DBV

Commit message: Kicad: PCB: x-2: use edge-cuts, rather than NPTH that sit on board's edge
Parts:
- removed H5, H6: MountingHole, lumberjack:MountingSlot_M2
Other:
- outline, holes or cut-outs redrawn

Commit message: Kicad: PCB: use 0.3mm via drill (via size 0.6mm) so that via >=0.15mm
For PCB Fabrication manufacturer SmartPCB88
Other:
- net class Default: via_drill 0.4 -> 0.3
- net class PWR: via_drill 0.4 -> 0.3
