File: pcb/keyboard-x2-lumberjack-arm.kicad_sch (KiCad schematic)
At the start: 141 parts, among them J1 16-pin USB-C Connector SMD, U1 STM32F103 Bluepill, or MiniF4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, U2 SN74LVC1T45DBV

Commit message: feat: 1U hotswap sw1-7 - sw1-12
Parts:
- SW_1_10, SW_1_11, SW_1_12, SW_1_7, SW_1_8, SW_1_9: footprint ProjectLocal:SW_MX_PG1350_NoLed -> ProjectLocal:MXOnly-1U-Hotswap-180
Changed lines of the file:
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@@
       (effects (font (size 1.27 1.27)) hide)
     )
-    (property "Footprint" "ProjectLocal:SW_MX_PG1350_NoLed" (id 2) (at 200.66 27.94 0)
+    (property "Footprint" "ProjectLocal:MXOnly-1U-Hotswap-180" (id 2) (at 200.66 27.94 0)
       (effects (font (size 1.27 1.27)) hide)
     )
@@
       (effects (font (size 1.27 1.27)) hide)
     )
-    (property "Footprint" "ProjectLocal:SW_MX_PG1350_NoLed" (id 2) (at 215.9 27.94 0)
+    (property "Footprint" "ProjectLocal:MXOnly-1U-Hotswap-180" (id 2) (at 215.9 27.94 0)
       (effects (font (size 1.27 1.27)) hide)
     )
@@
       (effects (font (size 1.27 1.27)) hide)
     )
-    (property "Footprint" "ProjectLocal:SW_MX_PG1350_NoLed" (id 2) (at 231.14 27.94 0)
+    (property "Footprint" "ProjectLocal:MXOnly-1U-Hotswap-180" (id 2) (at 231.14 27.94 0)
       (effects (font (size 1.27 1.27)) hide)
     )
@@
       (effects (font (size 1.27 1.27)) hide)
     )
-    (property "Footprint" "ProjectLocal:SW_MX_PG1350_NoLed" (id 2) (at 246.38 27.94 0)
+    (property "Footprint" "ProjectLocal:MXOnly-1U-Hotswap-180" (id 2) (at 246.38 27.94 0)
       (effects (font (size 1.27 1.27)) hide)
     )
@@
       (effects (font (size 1.27 1.27)) hide)
     )
-    (property "Footprint" "ProjectLocal:SW_MX_PG1350_NoLed" (id 2) (at 261.62 27.94 0)
+    (property "Footprint" "ProjectLocal:MXOnly-1U-Hotswap-180" (id 2) (at 261.62 27.94 0)
       (effects (font (size 1.27 1.27)) hide)
     )
@@
       (effects (font (size 1.27 1.27)) hide)
     )
-    (property "Footprint" "ProjectLocal:SW_MX_PG1350_NoLed" (id 2) (at 276.86 27.94 0)
+    (property "Footprint" "ProjectLocal:MXOnly-1U-Hotswap-180" (id 2) (at 276.86 27.94 0)
       (effects (font (size 1.27 1.27)) hide)
     )
@@
     )
     (path "/00000000-0000-0000-0000-000061d7d09b"
-      (reference "SW_1_7") (unit 1) (value "MX-compatible or Kailh Choc v1") (footprint "ProjectLocal:SW_MX_PG1350_NoLed")
+      (reference "SW_1_7") (unit 1) (value "MX-compatible or Kailh Choc v1") (footprint "ProjectLocal:MXOnly-1U-Hotswap-180")
     )
     (path "/00000000-0000-0000-0000-000061d81b29"
-      (reference "SW_1_8") (unit 1) (value "MX-compatible or Kailh Choc v1") (footprint "ProjectLocal:SW_MX_PG1350_NoLed")
+      (reference "SW_1_8") (unit 1) (value "MX-compatible or Kailh Choc v1") (footprint "ProjectLocal:MXOnly-1U-Hotswap-180")
     )
     (path "/00000000-0000-0000-0000-000061d8211a"
-      (reference "SW_1_9") (unit 1) (value "MX-compatible or Kailh Choc v1") (footprint "ProjectLocal:SW_MX_PG1350_NoLed")
+      (reference "SW_1_9") (unit 1) (value "MX-compatible or Kailh Choc v1") (footprint "ProjectLocal:MXOnly-1U-Hotswap-180")
     )
     (path "/00000000-0000-0000-0000-000061d82662"
-      (reference "SW_1_10") (unit 1) (value "MX-compatible or Kailh Choc v1") (footprint "ProjectLocal:SW_MX_PG1350_NoLed")
+      (reference "SW_1_10") (unit 1) (value "MX-compatible or Kailh Choc v1") (footprint "ProjectLocal:MXOnly-1U-Hotswap-180")
     )
     (path "/00000000-0000-0000-0000-000061d82b97"
-      (reference "SW_1_11") (unit 1) (value "MX-compatible or Kailh Choc v1") (footprint "ProjectLocal:SW_MX_PG1350_NoLed")
+      (reference "SW_1_11") (unit 1) (value "MX-compatible or Kailh Choc v1") (footprint "ProjectLocal:MXOnly-1U-Hotswap-180")
     )
     (path "/00000000-0000-0000-0000-000061d830be"
-      (reference "SW_1_12") (unit 1) (value "MX-compatible or Kailh Choc v1") (footprint "ProjectLocal:SW_MX_PG1350_NoLed")
+      (reference "SW_1_12") (unit 1) (value "MX-compatible or Kailh Choc v1") (footprint "ProjectLocal:MXOnly-1U-Hotswap-180")
     )
     (path "/00000000-0000-0000-0000-000061d83c48"

Commit message: feat: 1U hotswap sw2-1 - sw2-12
Parts:
- SW_2_1, SW_2_10, SW_2_11, SW_2_12, SW_2_2, SW_2_3, SW_2_4, SW_2_5, SW_2_6, SW_2_7, SW_2_8, SW_2_9: footprint ProjectLocal:SW_MX_PG1350_NoLed -> ProjectLocal:MXOnly-1U-Hotswap-180
Changed lines of the file:
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@@
       (effects (font (size 1.27 1.27)) hide)
     )
-    (property "Footprint" "ProjectLocal:SW_MX_PG1350_NoLed" (id 2) (at 109.22 44.45 0)
+    (property "Footprint" "ProjectLocal:MXOnly-1U-Hotswap-180" (id 2) (at 109.22 44.45 0)
       (effects (font (size 1.27 1.27)) hide)
     )
@@
       (effects (font (size 1.27 1.27)) hide)
     )
-    (property "Footprint" "ProjectLocal:SW_MX_PG1350_NoLed" (id 2) (at 124.46 44.45 0)
+    (property "Footprint" "ProjectLocal:MXOnly-1U-Hotswap-180" (id 2) (at 124.46 44.45 0)
       (effects (font (size 1.27 1.27)) hide)
     )
@@
       (effects (font (size 1.27 1.27)) hide)
     )
-    (property "Footprint" "ProjectLocal:SW_MX_PG1350_NoLed" (id 2) (at 139.7 44.45 0)
+    (property "Footprint" "ProjectLocal:MXOnly-1U-Hotswap-180" (id 2) (at 139.7 44.45 0)
       (effects (font (size 1.27 1.27)) hide)
     )
@@
       (effects (font (size 1.27 1.27)) hide)
     )
-    (property "Footprint" "ProjectLocal:SW_MX_PG1350_NoLed" (id 2) (at 154.94 44.45 0)
+    (property "Footprint" "ProjectLocal:MXOnly-1U-Hotswap-180" (id 2) (at 154.94 44.45 0)
       (effects (font (size 1.27 1.27)) hide)
     )
@@
       (effects (font (size 1.27 1.27)) hide)
     )
-    (property "Footprint" "ProjectLocal:SW_MX_PG1350_NoLed" (id 2) (at 170.18 44.45 0)
+    (property "Footprint" "ProjectLocal:MXOnly-1U-Hotswap-180" (id 2) (at 170.18 44.45 0)
       (effects (font (size 1.27 1.27)) hide)
     )
@@
       (effects (font (size 1.27 1.27)) hide)
     )
-    (property "Footprint" "ProjectLocal:SW_MX_PG1350_NoLed" (id 2) (at 185.42 44.45 0)
+    (property "Footprint" "ProjectLocal:MXOnly-1U-Hotswap-180" (id 2) (at 185.42 44.45 0)
       (effects (font (size 1.27 1.27)) hide)
     )
@@
       (effects (font (size 1.27 1.27)) hide)
     )
-    (property "Footprint" "ProjectLocal:SW_MX_PG1350_NoLed" (id 2) (at 200.66 44.45 0)
+    (property "Footprint" "ProjectLocal:MXOnly-1U-Hotswap-180" (id 2) (at 200.66 44.45 0)
       (effects (font (size 1.27 1.27)) hide)
     )
@@
       (effects (font (size 1.27 1.27)) hide)
     )
-    (property "Footprint" "ProjectLocal:SW_MX_PG1350_NoLed" (id 2) (at 215.9 44.45 0)
+    (property "Footprint" "ProjectLocal:MXOnly-1U-Hotswap-180" (id 2) (at 215.9 44.45 0)
       (effects (font (size 1.27 1.27)) hide)
     )
@@
       (effects (font (size 1.27 1.27)) hide)
     )
-    (property "Footprint" "ProjectLocal:SW_MX_PG1350_NoLed" (id 2) (at 231.14 44.45 0)
+    (property "Footprint" "ProjectLocal:MXOnly-1U-Hotswap-180" (id 2) (at 231.14 44.45 0)
       (effects (font (size 1.27 1.27)) hide)
     )
@@
       (effects (font (size 1.27 1.27)) hide)
     )
-    (property "Footprint" "ProjectLocal:SW_MX_PG1350_NoLed" (id 2) (at 246.38 44.45 0)
+    (property "Footprint" "ProjectLocal:MXOnly-1U-Hotswap-180" (id 2) (at 246.38 44.45 0)
       (effects (font (size 1.27 1.27)) hide)
     )
@@
       (effects (font (size 1.27 1.27)) hide)
     )
-    (property "Footprint" "ProjectLocal:SW_MX_PG1350_NoLed" (id 2) (at 261.62 44.45 0)
+    (property "Footprint" "ProjectLocal:MXOnly-1U-Hotswap-180" (id 2) (at 261.62 44.45 0)
       (effects (font (size 1.27 1.27)) hide)
     )
@@
       (effects (font (size 1.27 1.27)) hide)
     )
-    (property "Footprint" "ProjectLocal:SW_MX_PG1350_NoLed" (id 2) (at 276.86 44.45 0)
+    (property "Footprint" "ProjectLocal:MXOnly-1U-Hotswap-180" (id 2) (at 276.86 44.45 0)
       (effects (font (size 1.27 1.27)) hide)
     )
@@
     )
     (path "/00000000-0000-0000-0000-000061d83c48"
-      (reference "SW_2_1") (unit 1) (value "MX-compatible or Kailh Choc v1") (footprint "ProjectLocal:SW_MX_PG1350_NoLed")
+      (reference "SW_2_1") (unit 1) (value "MX-compatible or Kailh Choc v1") (footprint "ProjectLocal:MXOnly-1U-Hotswap-180")
     )
     (path "/00000000-0000-0000-0000-000061d8c34b"
-      (reference "SW_2_2") (unit 1) (value "MX-compatible or Kailh Choc v1") (footprint "ProjectLocal:SW_MX_PG1350_NoLed")
+      (reference "SW_2_2") (unit 1) (value "MX-compatible or Kailh Choc v1") (footprint "ProjectLocal:MXOnly-1U-Hotswap-180")
     )
     (path "/00000000-0000-0000-0000-000061d8c7b7"
-      (reference "SW_2_3") (unit 1) (value "MX-compatible or Kailh Choc v1") (footprint "ProjectLocal:SW_MX_PG1350_NoLed")
+      (reference "SW_2_3") (unit 1) (value "MX-compatible or Kailh Choc v1") (footprint "ProjectLocal:MXOnly-1U-Hotswap-180")
     )
     (path "/00000000-0000-0000-0000-000061d8cbf6"
-      (reference "SW_2_4") (unit 1) (value "MX-compatible or Kailh Choc v1") (footprint "ProjectLocal:SW_MX_PG1350_NoLed")
+      (reference "SW_2_4") (unit 1) (value "MX-compatible or Kailh Choc v1") (footprint "ProjectLocal:MXOnly-1U-Hotswap-180")
     )
     (path "/00000000-0000-0000-0000-000061d8d158"
-      (reference "SW_2_5") (unit 1) (value "MX-compatible or Kailh Choc v1") (footprint "ProjectLocal:SW_MX_PG1350_NoLed")
+      (reference "SW_2_5") (unit 1) (value "MX-compatible or Kailh Choc v1") (footprint "ProjectLocal:MXOnly-1U-Hotswap-180")
     )
     (path "/00000000-0000-0000-0000-000061d8d561"
-      (reference "SW_2_6") (unit 1) (value "MX-compatible or Kailh Choc v1") (footprint "ProjectLocal:SW_MX_PG1350_NoLed")
+      (reference "SW_2_6") (unit 1) (value "MX-compatible or Kailh Choc v1") (footprint "ProjectLocal:MXOnly-1U-Hotswap-180")
     )
     (path "/00000000-0000-0000-0000-000061d8da83"
-      (reference "SW_2_7") (unit 1) (value "MX-compatible or Kailh Choc v1") (footprint "ProjectLocal:SW_MX_PG1350_NoLed")
+      (reference "SW_2_7") (unit 1) (value "MX-compatible or Kailh Choc v1") (footprint "ProjectLocal:MXOnly-1U-Hotswap-180")
     )
     (path "/00000000-0000-0000-0000-000061d8e07e"
-      (reference "SW_2_8") (unit 1) (value "MX-compatible or Kailh Choc v1") (footprint "ProjectLocal:SW_MX_PG1350_NoLed")
+      (reference "SW_2_8") (unit 1) (value "MX-compatible or Kailh Choc v1") (footprint "ProjectLocal:MXOnly-1U-Hotswap-180")
     )
     (path "/00000000-0000-0000-0000-000061d8e636"
-      (reference "SW_2_9") (unit 1) (value "MX-compatible or Kailh Choc v1") (footprint "ProjectLocal:SW_MX_PG1350_NoLed")
+      (reference "SW_2_9") (unit 1) (value "MX-compatible or Kailh Choc v1") (footprint "ProjectLocal:MXOnly-1U-Hotswap-180")
     )
     (path "/00000000-0000-0000-0000-000061d8eb73"
-      (reference "SW_2_10") (unit 1) (value "MX-compatible or Kailh Choc v1") (footprint "ProjectLocal:SW_MX_PG1350_NoLed")
+      (reference "SW_2_10") (unit 1) (value "MX-compatible or Kailh Choc v1") (footprint "ProjectLocal:MXOnly-1U-Hotswap-180")
     )
     (path "/00000000-0000-0000-0000-000061d8eed1"
-      (reference "SW_2_11") (unit 1) (value "MX-compatible or Kailh Choc v1") (footprint "ProjectLocal:SW_MX_PG1350_NoLed")
+      (reference "SW_2_11") (unit 1) (value "MX-compatible or Kailh Choc v1") (footprint "ProjectLocal:MXOnly-1U-Hotswap-180")
     )
     (path "/00000000-0000-0000-0000-000061d8f4c9"
-      (reference "SW_2_12") (unit 1) (value "MX-compatible or Kailh Choc v1") (footprint "ProjectLocal:SW_MX_PG1350_NoLed")
+      (reference "SW_2_12") (unit 1) (value "MX-compatible or Kailh Choc v1") (footprint "ProjectLocal:MXOnly-1U-Hotswap-180")
     )
     (path "/00000000-0000-0000-0000-000061d866dc"

Commit message: feat: 1U hotswap sw3-1 - sw3-12
Parts:
- SW_3_1, SW_3_10, SW_3_11, SW_3_12, SW_3_2, SW_3_3, SW_3_4, SW_3_5, SW_3_6, SW_3_7, SW_3_8, SW_3_9: footprint ProjectLocal:SW_MX_PG1350_NoLed -> ProjectLocal:MXOnly-1U-Hotswap-180
Changed lines of the file:
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@@
       (effects (font (size 1.27 1.27)) hide)
     )
-    (property "Footprint" "ProjectLocal:SW_MX_PG1350_NoLed" (id 2) (at 109.22 60.96 0)
+    (property "Footprint" "ProjectLocal:MXOnly-1U-Hotswap-180" (id 2) (at 109.22 60.96 0)
       (effects (font (size 1.27 1.27)) hide)
     )
@@
       (effects (font (size 1.27 1.27)) hide)
     )
-    (property "Footprint" "ProjectLocal:SW_MX_PG1350_NoLed" (id 2) (at 124.46 60.96 0)
+    (property "Footprint" "ProjectLocal:MXOnly-1U-Hotswap-180" (id 2) (at 124.46 60.96 0)
       (effects (font (size 1.27 1.27)) hide)
     )
@@
       (effects (font (size 1.27 1.27)) hide)
     )
-    (property "Footprint" "ProjectLocal:SW_MX_PG1350_NoLed" (id 2) (at 139.7 60.96 0)
+    (property "Footprint" "ProjectLocal:MXOnly-1U-Hotswap-180" (id 2) (at 139.7 60.96 0)
       (effects (font (size 1.27 1.27)) hide)
     )
@@
       (effects (font (size 1.27 1.27)) hide)
     )
-    (property "Footprint" "ProjectLocal:SW_MX_PG1350_NoLed" (id 2) (at 154.94 60.96 0)
+    (property "Footprint" "ProjectLocal:MXOnly-1U-Hotswap-180" (id 2) (at 154.94 60.96 0)
       (effects (font (size 1.27 1.27)) hide)
     )
@@
       (effects (font (size 1.27 1.27)) hide)
     )
-    (property "Footprint" "ProjectLocal:SW_MX_PG1350_NoLed" (id 2) (at 170.18 60.96 0)
+    (property "Footprint" "ProjectLocal:MXOnly-1U-Hotswap-180" (id 2) (at 170.18 60.96 0)
       (effects (font (size 1.27 1.27)) hide)
     )
@@
       (effects (font (size 1.27 1.27)) hide)
     )
-    (property "Footprint" "ProjectLocal:SW_MX_PG1350_NoLed" (id 2) (at 185.42 60.96 0)
+    (property "Footprint" "ProjectLocal:MXOnly-1U-Hotswap-180" (id 2) (at 185.42 60.96 0)
       (effects (font (size 1.27 1.27)) hide)
     )
@@
       (effects (font (size 1.27 1.27)) hide)
     )
-    (property "Footprint" "ProjectLocal:SW_MX_PG1350_NoLed" (id 2) (at 200.66 60.96 0)
+    (property "Footprint" "ProjectLocal:MXOnly-1U-Hotswap-180" (id 2) (at 200.66 60.96 0)
       (effects (font (size 1.27 1.27)) hide)
     )
@@
       (effects (font (size 1.27 1.27)) hide)
     )
-    (property "Footprint" "ProjectLocal:SW_MX_PG1350_NoLed" (id 2) (at 215.9 60.96 0)
+    (property "Footprint" "ProjectLocal:MXOnly-1U-Hotswap-180" (id 2) (at 215.9 60.96 0)
       (effects (font (size 1.27 1.27)) hide)
     )
@@
       (effects (font (size 1.27 1.27)) hide)
     )
-    (property "Footprint" "ProjectLocal:SW_MX_PG1350_NoLed" (id 2) (at 231.14 60.96 0)
+    (property "Footprint" "ProjectLocal:MXOnly-1U-Hotswap-180" (id 2) (at 231.14 60.96 0)
       (effects (font (size 1.27 1.27)) hide)
     )
@@
       (effects (font (size 1.27 1.27)) hide)
     )
-    (property "Footprint" "ProjectLocal:SW_MX_PG1350_NoLed" (id 2) (at 246.38 60.96 0)
+    (property "Footprint" "ProjectLocal:MXOnly-1U-Hotswap-180" (id 2) (at 246.38 60.96 0)
       (effects (font (size 1.27 1.27)) hide)
     )
@@
       (effects (font (size 1.27 1.27)) hide)
     )
-    (property "Footprint" "ProjectLocal:SW_MX_PG1350_NoLed" (id 2) (at 261.62 60.96 0)
+    (property "Footprint" "ProjectLocal:MXOnly-1U-Hotswap-180" (id 2) (at 261.62 60.96 0)
       (effects (font (size 1.27 1.27)) hide)
     )
@@
       (effects (font (size 1.27 1.27)) hide)
     )
-    (property "Footprint" "ProjectLocal:SW_MX_PG1350_NoLed" (id 2) (at 276.86 60.96 0)
+    (property "Footprint" "ProjectLocal:MXOnly-1U-Hotswap-180" (id 2) (at 276.86 60.96 0)
       (effects (font (size 1.27 1.27)) hide)
     )
@@
     )
     (path "/00000000-0000-0000-0000-000061d866dc"
-      (reference "SW_3_1") (unit 1) (value "MX-compatible or Kailh Choc v1") (footprint "ProjectLocal:SW_MX_PG1350_NoLed")
+      (reference "SW_3_1") (unit 1) (value "MX-compatible or Kailh Choc v1") (footprint "ProjectLocal:MXOnly-1U-Hotswap-180")
     )
     (path "/00000000-0000-0000-0000-000061d8f986"
-      (reference "SW_3_2") (unit 1) (value "MX-compatible or Kailh Choc v1") (footprint "ProjectLocal:SW_MX_PG1350_NoLed")
+      (reference "SW_3_2") (unit 1) (value "MX-compatible or Kailh Choc v1") (footprint "ProjectLocal:MXOnly-1U-Hotswap-180")
     )
     (path "/00000000-0000-0000-0000-000061d8fe94"
-      (reference "SW_3_3") (unit 1) (value "MX-compatible or Kailh Choc v1") (footprint "ProjectLocal:SW_MX_PG1350_NoLed")
+      (reference "SW_3_3") (unit 1) (value "MX-compatible or Kailh Choc v1") (footprint "ProjectLocal:MXOnly-1U-Hotswap-180")
     )
     (path "/00000000-0000-0000-0000-000061d902b3"
-      (reference "SW_3_4") (unit 1) (value "MX-compatible or Kailh Choc v1") (footprint "ProjectLocal:SW_MX_PG1350_NoLed")
+      (reference "SW_3_4") (unit 1) (value "MX-compatible or Kailh Choc v1") (footprint "ProjectLocal:MXOnly-1U-Hotswap-180")
     )
     (path "/00000000-0000-0000-0000-000061d909ac"
-      (reference "SW_3_5") (unit 1) (value "MX-compatible or Kailh Choc v1") (footprint "ProjectLocal:SW_MX_PG1350_NoLed")
+      (reference "SW_3_5") (unit 1) (value "MX-compatible or Kailh Choc v1") (footprint "ProjectLocal:MXOnly-1U-Hotswap-180")
     )
     (path "/00000000-0000-0000-0000-000061d911ad"
-      (reference "SW_3_6") (unit 1) (value "MX-compatible or Kailh Choc v1") (footprint "ProjectLocal:SW_MX_PG1350_NoLed")
+      (reference "SW_3_6") (unit 1) (value "MX-compatible or Kailh Choc v1") (footprint "ProjectLocal:MXOnly-1U-Hotswap-180")
     )
     (path "/00000000-0000-0000-0000-000061db90d1"
-      (reference "SW_3_7") (unit 1) (value "MX-compatible or Kailh Choc v1") (footprint "ProjectLocal:SW_MX_PG1350_NoLed")
+      (reference "SW_3_7") (unit 1) (value "MX-compatible or Kailh Choc v1") (footprint "ProjectLocal:MXOnly-1U-Hotswap-180")
     )
     (path "/00000000-0000-0000-0000-000061db96fe"
-      (reference "SW_3_8") (unit 1) (value "MX-compatible or Kailh Choc v1") (footprint "ProjectLocal:SW_MX_PG1350_NoLed")
+      (reference "SW_3_8") (unit 1) (value "MX-compatible or Kailh Choc v1") (footprint "ProjectLocal:MXOnly-1U-Hotswap-180")
     )
     (path "/00000000-0000-0000-0000-000061db9db5"
-      (reference "SW_3_9") (unit 1) (value "MX-compatible or Kailh Choc v1") (footprint "ProjectLocal:SW_MX_PG1350_NoLed")
+      (reference "SW_3_9") (unit 1) (value "MX-compatible or Kailh Choc v1") (footprint "ProjectLocal:MXOnly-1U-Hotswap-180")
     )
     (path "/00000000-0000-0000-0000-000061dba30d"
-      (reference "SW_3_10") (unit 1) (value "MX-compatible or Kailh Choc v1") (footprint "ProjectLocal:SW_MX_PG1350_NoLed")
+      (reference "SW_3_10") (unit 1) (value "MX-compatible or Kailh Choc v1") (footprint "ProjectLocal:MXOnly-1U-Hotswap-180")
     )
     (path "/00000000-0000-0000-0000-000061dba7ac"
-      (reference "SW_3_11") (unit 1) (value "MX-compatible or Kailh Choc v1") (footprint "ProjectLocal:SW_MX_PG1350_NoLed")
+      (reference "SW_3_11") (unit 1) (value "MX-compatible or Kailh Choc v1") (footprint "ProjectLocal:MXOnly-1U-Hotswap-180")
     )
     (path "/00000000-0000-0000-0000-000061dbad55"
-      (reference "SW_3_12") (unit 1) (value "MX-compatible or Kailh Choc v1") (footprint "ProjectLocal:SW_MX_PG1350_NoLed")
+      (reference "SW_3_12") (unit 1) (value "MX-compatible or Kailh Choc v1") (footprint "ProjectLocal:MXOnly-1U-Hotswap-180")
     )
     (path "/00000000-0000-0000-0000-000061d87edc"
