File: pcb/keyboard-x2-lumberjack-arm.kicad_sch (KiCad schematic)
At the start: 141 parts, among them J1 16-pin USB-C Connector SMD, U1 STM32F103 Bluepill, or MiniF4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, U2 SN74LVC1T45DBV

Commit message: feat: 1U hotswap sw4-1 - sw4-12
Parts:
- SW_4_1, SW_4_10, SW_4_11, SW_4_12, SW_4_2, SW_4_3, SW_4_4, SW_4_5, SW_4_6, SW_4_7, SW_4_8, SW_4_9: footprint ProjectLocal:SW_MX_PG1350_NoLed -> ProjectLocal:MXOnly-1U-Hotswap-180
Changed lines of the file:
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@@
       (effects (font (size 1.27 1.27)) hide)
     )
-    (property "Footprint" "ProjectLocal:SW_MX_PG1350_NoLed" (id 2) (at 109.22 77.47 0)
+    (property "Footprint" "ProjectLocal:MXOnly-1U-Hotswap-180" (id 2) (at 109.22 77.47 0)
       (effects (font (size 1.27 1.27)) hide)
     )
@@
       (effects (font (size 1.27 1.27)) hide)
     )
-    (property "Footprint" "ProjectLocal:SW_MX_PG1350_NoLed" (id 2) (at 124.46 77.47 0)
+    (property "Footprint" "ProjectLocal:MXOnly-1U-Hotswap-180" (id 2) (at 124.46 77.47 0)
       (effects (font (size 1.27 1.27)) hide)
     )
@@
       (effects (font (size 1.27 1.27)) hide)
     )
-    (property "Footprint" "ProjectLocal:SW_MX_PG1350_NoLed" (id 2) (at 139.7 77.47 0)
+    (property "Footprint" "ProjectLocal:MXOnly-1U-Hotswap-180" (id 2) (at 139.7 77.47 0)
       (effects (font (size 1.27 1.27)) hide)
     )
@@
       (effects (font (size 1.27 1.27)) hide)
     )
-    (property "Footprint" "ProjectLocal:SW_MX_PG1350_NoLed" (id 2) (at 154.94 77.47 0)
+    (property "Footprint" "ProjectLocal:MXOnly-1U-Hotswap-180" (id 2) (at 154.94 77.47 0)
       (effects (font (size 1.27 1.27)) hide)
     )
@@
       (effects (font (size 1.27 1.27)) hide)
     )
-    (property "Footprint" "ProjectLocal:SW_MX_PG1350_NoLed" (id 2) (at 170.18 77.47 0)
+    (property "Footprint" "ProjectLocal:MXOnly-1U-Hotswap-180" (id 2) (at 170.18 77.47 0)
       (effects (font (size 1.27 1.27)) hide)
     )
@@
       (effects (font (size 1.27 1.27)) hide)
     )
-    (property "Footprint" "ProjectLocal:SW_MX_PG1350_NoLed" (id 2) (at 185.42 77.47 0)
+    (property "Footprint" "ProjectLocal:MXOnly-1U-Hotswap-180" (id 2) (at 185.42 77.47 0)
       (effects (font (size 1.27 1.27)) hide)
     )
@@
       (effects (font (size 1.27 1.27)) hide)
     )
-    (property "Footprint" "ProjectLocal:SW_MX_PG1350_NoLed" (id 2) (at 200.66 77.47 0)
+    (property "Footprint" "ProjectLocal:MXOnly-1U-Hotswap-180" (id 2) (at 200.66 77.47 0)
       (effects (font (size 1.27 1.27)) hide)
     )
@@
       (effects (font (size 1.27 1.27)) hide)
     )
-    (property "Footprint" "ProjectLocal:SW_MX_PG1350_NoLed" (id 2) (at 215.9 77.47 0)
+    (property "Footprint" "ProjectLocal:MXOnly-1U-Hotswap-180" (id 2) (at 215.9 77.47 0)
       (effects (font (size 1.27 1.27)) hide)
     )
@@
       (effects (font (size 1.27 1.27)) hide)
     )
-    (property "Footprint" "ProjectLocal:SW_MX_PG1350_NoLed" (id 2) (at 231.14 77.47 0)
+    (property "Footprint" "ProjectLocal:MXOnly-1U-Hotswap-180" (id 2) (at 231.14 77.47 0)
       (effects (font (size 1.27 1.27)) hide)
     )
@@
       (effects (font (size 1.27 1.27)) hide)
     )
-    (property "Footprint" "ProjectLocal:SW_MX_PG1350_NoLed" (id 2) (at 246.38 77.47 0)
+    (property "Footprint" "ProjectLocal:MXOnly-1U-Hotswap-180" (id 2) (at 246.38 77.47 0)
       (effects (font (size 1.27 1.27)) hide)
     )
@@
       (effects (font (size 1.27 1.27)) hide)
     )
-    (property "Footprint" "ProjectLocal:SW_MX_PG1350_NoLed" (id 2) (at 261.62 77.47 0)
+    (property "Footprint" "ProjectLocal:MXOnly-1U-Hotswap-180" (id 2) (at 261.62 77.47 0)
       (effects (font (size 1.27 1.27)) hide)
     )
@@
       (effects (font (size 1.27 1.27)) hide)
     )
-    (property "Footprint" "ProjectLocal:SW_MX_PG1350_NoLed" (id 2) (at 276.86 77.47 0)
+    (property "Footprint" "ProjectLocal:MXOnly-1U-Hotswap-180" (id 2) (at 276.86 77.47 0)
       (effects (font (size 1.27 1.27)) hide)
     )
@@
     )
     (path "/00000000-0000-0000-0000-000061d87edc"
-      (reference "SW_4_1") (unit 1) (value "MX-compatible or Kailh Choc v1") (footprint "ProjectLocal:SW_MX_PG1350_NoLed")
+      (reference "SW_4_1") (unit 1) (value "MX-compatible or Kailh Choc v1") (footprint "ProjectLocal:MXOnly-1U-Hotswap-180")
     )
     (path "/00000000-0000-0000-0000-000061dc180a"
-      (reference "SW_4_2") (unit 1) (value "MX-compatible or Kailh Choc v1") (footprint "ProjectLocal:SW_MX_PG1350_NoLed")
+      (reference "SW_4_2") (unit 1) (value "MX-compatible or Kailh Choc v1") (footprint "ProjectLocal:MXOnly-1U-Hotswap-180")
     )
     (path "/00000000-0000-0000-0000-000061dc1d4b"
-      (reference "SW_4_3") (unit 1) (value "MX-compatible or Kailh Choc v1") (footprint "ProjectLocal:SW_MX_PG1350_NoLed")
+      (reference "SW_4_3") (unit 1) (value "MX-compatible or Kailh Choc v1") (footprint "ProjectLocal:MXOnly-1U-Hotswap-180")
     )
     (path "/00000000-0000-0000-0000-000061dc218f"
-      (reference "SW_4_4") (unit 1) (value "MX-compatible or Kailh Choc v1") (footprint "ProjectLocal:SW_MX_PG1350_NoLed")
+      (reference "SW_4_4") (unit 1) (value "MX-compatible or Kailh Choc v1") (footprint "ProjectLocal:MXOnly-1U-Hotswap-180")
     )
     (path "/00000000-0000-0000-0000-000061dc24b1"
-      (reference "SW_4_5") (unit 1) (value "MX-compatible or Kailh Choc v1") (footprint "ProjectLocal:SW_MX_PG1350_NoLed")
+      (reference "SW_4_5") (unit 1) (value "MX-compatible or Kailh Choc v1") (footprint "ProjectLocal:MXOnly-1U-Hotswap-180")
     )
     (path "/00000000-0000-0000-0000-000061dc28f0"
-      (reference "SW_4_6") (unit 1) (value "MX-compatible or Kailh Choc v1") (footprint "ProjectLocal:SW_MX_PG1350_NoLed")
+      (reference "SW_4_6") (unit 1) (value "MX-compatible or Kailh Choc v1") (footprint "ProjectLocal:MXOnly-1U-Hotswap-180")
     )
     (path "/00000000-0000-0000-0000-000061dc2e93"
-      (reference "SW_4_7") (unit 1) (value "MX-compatible or Kailh Choc v1") (footprint "ProjectLocal:SW_MX_PG1350_NoLed")
+      (reference "SW_4_7") (unit 1) (value "MX-compatible or Kailh Choc v1") (footprint "ProjectLocal:MXOnly-1U-Hotswap-180")
     )
     (path "/00000000-0000-0000-0000-000061dc3742"
-      (reference "SW_4_8") (unit 1) (value "MX-compatible or Kailh Choc v1") (footprint "ProjectLocal:SW_MX_PG1350_NoLed")
+      (reference "SW_4_8") (unit 1) (value "MX-compatible or Kailh Choc v1") (footprint "ProjectLocal:MXOnly-1U-Hotswap-180")
     )
     (path "/00000000-0000-0000-0000-000061dc3e43"
-      (reference "SW_4_9") (unit 1) (value "MX-compatible or Kailh Choc v1") (footprint "ProjectLocal:SW_MX_PG1350_NoLed")
+      (reference "SW_4_9") (unit 1) (value "MX-compatible or Kailh Choc v1") (footprint "ProjectLocal:MXOnly-1U-Hotswap-180")
     )
     (path "/00000000-0000-0000-0000-000061dc4302"
-      (reference "SW_4_10") (unit 1) (value "MX-compatible or Kailh Choc v1") (footprint "ProjectLocal:SW_MX_PG1350_NoLed")
+      (reference "SW_4_10") (unit 1) (value "MX-compatible or Kailh Choc v1") (footprint "ProjectLocal:MXOnly-1U-Hotswap-180")
     )
     (path "/00000000-0000-0000-0000-000061dc49b4"
-      (reference "SW_4_11") (unit 1) (value "MX-compatible or Kailh Choc v1") (footprint "ProjectLocal:SW_MX_PG1350_NoLed")
+      (reference "SW_4_11") (unit 1) (value "MX-compatible or Kailh Choc v1") (footprint "ProjectLocal:MXOnly-1U-Hotswap-180")
     )
     (path "/00000000-0000-0000-0000-000061dc4dc5"
-      (reference "SW_4_12") (unit 1) (value "MX-compatible or Kailh Choc v1") (footprint "ProjectLocal:SW_MX_PG1350_NoLed")
+      (reference "SW_4_12") (unit 1) (value "MX-compatible or Kailh Choc v1") (footprint "ProjectLocal:MXOnly-1U-Hotswap-180")
     )
     (path "/00000000-0000-0000-0000-000061d88593"

Commit message: feat: 1U hotswap sw5-1 - sw5-12
Parts:
- SW_5_1, SW_5_10, SW_5_11, SW_5_12, SW_5_2, SW_5_3, SW_5_4, SW_5_5, SW_5_6, SW_5_7, SW_5_8, SW_5_9: footprint ProjectLocal:SW_MX_PG1350_NoLed -> ProjectLocal:MXOnly-1U-Hotswap-180
Changed lines of the file:
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@@
       (effects (font (size 1.27 1.27)) hide)
     )
-    (property "Footprint" "ProjectLocal:SW_MX_PG1350_NoLed" (id 2) (at 109.22 93.98 0)
+    (property "Footprint" "ProjectLocal:MXOnly-1U-Hotswap-180" (id 2) (at 109.22 93.98 0)
       (effects (font (size 1.27 1.27)) hide)
     )
@@
       (effects (font (size 1.27 1.27)) hide)
     )
-    (property "Footprint" "ProjectLocal:SW_MX_PG1350_NoLed" (id 2) (at 124.46 93.98 0)
+    (property "Footprint" "ProjectLocal:MXOnly-1U-Hotswap-180" (id 2) (at 124.46 93.98 0)
       (effects (font (size 1.27 1.27)) hide)
     )
@@
       (effects (font (size 1.27 1.27)) hide)
     )
-    (property "Footprint" "ProjectLocal:SW_MX_PG1350_NoLed" (id 2) (at 139.7 93.98 0)
+    (property "Footprint" "ProjectLocal:MXOnly-1U-Hotswap-180" (id 2) (at 139.7 93.98 0)
       (effects (font (size 1.27 1.27)) hide)
     )
@@
       (effects (font (size 1.27 1.27)) hide)
     )
-    (property "Footprint" "ProjectLocal:SW_MX_PG1350_NoLed" (id 2) (at 154.94 93.98 0)
+    (property "Footprint" "ProjectLocal:MXOnly-1U-Hotswap-180" (id 2) (at 154.94 93.98 0)
       (effects (font (size 1.27 1.27)) hide)
     )
@@
       (effects (font (size 1.27 1.27)) hide)
     )
-    (property "Footprint" "ProjectLocal:SW_MX_PG1350_NoLed" (id 2) (at 170.18 93.98 0)
+    (property "Footprint" "ProjectLocal:MXOnly-1U-Hotswap-180" (id 2) (at 170.18 93.98 0)
       (effects (font (size 1.27 1.27)) hide)
     )
@@
       (effects (font (size 1.27 1.27)) hide)
     )
-    (property "Footprint" "ProjectLocal:SW_MX_PG1350_NoLed" (id 2) (at 185.42 93.98 0)
+    (property "Footprint" "ProjectLocal:MXOnly-1U-Hotswap-180" (id 2) (at 185.42 93.98 0)
       (effects (font (size 1.27 1.27)) hide)
     )
@@
       (effects (font (size 1.27 1.27)) hide)
     )
-    (property "Footprint" "ProjectLocal:SW_MX_PG1350_NoLed" (id 2) (at 200.66 93.98 0)
+    (property "Footprint" "ProjectLocal:MXOnly-1U-Hotswap-180" (id 2) (at 200.66 93.98 0)
       (effects (font (size 1.27 1.27)) hide)
     )
@@
       (effects (font (size 1.27 1.27)) hide)
     )
-    (property "Footprint" "ProjectLocal:SW_MX_PG1350_NoLed" (id 2) (at 215.9 93.98 0)
+    (property "Footprint" "ProjectLocal:MXOnly-1U-Hotswap-180" (id 2) (at 215.9 93.98 0)
       (effects (font (size 1.27 1.27)) hide)
     )
@@
       (effects (font (size 1.27 1.27)) hide)
     )
-    (property "Footprint" "ProjectLocal:SW_MX_PG1350_NoLed" (id 2) (at 231.14 93.98 0)
+    (property "Footprint" "ProjectLocal:MXOnly-1U-Hotswap-180" (id 2) (at 231.14 93.98 0)
       (effects (font (size 1.27 1.27)) hide)
     )
@@
       (effects (font (size 1.27 1.27)) hide)
     )
-    (property "Footprint" "ProjectLocal:SW_MX_PG1350_NoLed" (id 2) (at 246.38 93.98 0)
+    (property "Footprint" "ProjectLocal:MXOnly-1U-Hotswap-180" (id 2) (at 246.38 93.98 0)
       (effects (font (size 1.27 1.27)) hide)
     )
@@
       (effects (font (size 1.27 1.27)) hide)
     )
-    (property "Footprint" "ProjectLocal:SW_MX_PG1350_NoLed" (id 2) (at 261.62 93.98 0)
+    (property "Footprint" "ProjectLocal:MXOnly-1U-Hotswap-180" (id 2) (at 261.62 93.98 0)
       (effects (font (size 1.27 1.27)) hide)
     )
@@
       (effects (font (size 1.27 1.27)) hide)
     )
-    (property "Footprint" "ProjectLocal:SW_MX_PG1350_NoLed" (id 2) (at 276.86 93.98 0)
+    (property "Footprint" "ProjectLocal:MXOnly-1U-Hotswap-180" (id 2) (at 276.86 93.98 0)
       (effects (font (size 1.27 1.27)) hide)
     )
@@
     )
     (path "/00000000-0000-0000-0000-000061d88593"
-      (reference "SW_5_1") (unit 1) (value "MX-compatible or Kailh Choc v1") (footprint "ProjectLocal:SW_MX_PG1350_NoLed")
+      (reference "SW_5_1") (unit 1) (value "MX-compatible or Kailh Choc v1") (footprint "ProjectLocal:MXOnly-1U-Hotswap-180")
     )
     (path "/00000000-0000-0000-0000-000061dc530e"
-      (reference "SW_5_2") (unit 1) (value "MX-compatible or Kailh Choc v1") (footprint "ProjectLocal:SW_MX_PG1350_NoLed")
+      (reference "SW_5_2") (unit 1) (value "MX-compatible or Kailh Choc v1") (footprint "ProjectLocal:MXOnly-1U-Hotswap-180")
     )
     (path "/00000000-0000-0000-0000-000061dc5a7e"
-      (reference "SW_5_3") (unit 1) (value "MX-compatible or Kailh Choc v1") (footprint "ProjectLocal:SW_MX_PG1350_NoLed")
+      (reference "SW_5_3") (unit 1) (value "MX-compatible or Kailh Choc v1") (footprint "ProjectLocal:MXOnly-1U-Hotswap-180")
     )
     (path "/00000000-0000-0000-0000-000061dc600b"
-      (reference "SW_5_4") (unit 1) (value "MX-compatible or Kailh Choc v1") (footprint "ProjectLocal:SW_MX_PG1350_NoLed")
+      (reference "SW_5_4") (unit 1) (value "MX-compatible or Kailh Choc v1") (footprint "ProjectLocal:MXOnly-1U-Hotswap-180")
     )
     (path "/00000000-0000-0000-0000-000061dc6332"
-      (reference "SW_5_5") (unit 1) (value "MX-compatible or Kailh Choc v1") (footprint "ProjectLocal:SW_MX_PG1350_NoLed")
+      (reference "SW_5_5") (unit 1) (value "MX-compatible or Kailh Choc v1") (footprint "ProjectLocal:MXOnly-1U-Hotswap-180")
     )
     (path "/00000000-0000-0000-0000-000061dc698e"
-      (reference "SW_5_6") (unit 1) (value "MX-compatible or Kailh Choc v1") (footprint "ProjectLocal:SW_MX_PG1350_NoLed")
+      (reference "SW_5_6") (unit 1) (value "MX-compatible or Kailh Choc v1") (footprint "ProjectLocal:MXOnly-1U-Hotswap-180")
     )
     (path "/00000000-0000-0000-0000-000061dc6dcb"
-      (reference "SW_5_7") (unit 1) (value "MX-compatible or Kailh Choc v1") (footprint "ProjectLocal:SW_MX_PG1350_NoLed")
+      (reference "SW_5_7") (unit 1) (value "MX-compatible or Kailh Choc v1") (footprint "ProjectLocal:MXOnly-1U-Hotswap-180")
     )
     (path "/00000000-0000-0000-0000-000061dc7243"
-      (reference "SW_5_8") (unit 1) (value "MX-compatible or Kailh Choc v1") (footprint "ProjectLocal:SW_MX_PG1350_NoLed")
+      (reference "SW_5_8") (unit 1) (value "MX-compatible or Kailh Choc v1") (footprint "ProjectLocal:MXOnly-1U-Hotswap-180")
     )
     (path "/00000000-0000-0000-0000-000061dc77a2"
-      (reference "SW_5_9") (unit 1) (value "MX-compatible or Kailh Choc v1") (footprint "ProjectLocal:SW_MX_PG1350_NoLed")
+      (reference "SW_5_9") (unit 1) (value "MX-compatible or Kailh Choc v1") (footprint "ProjectLocal:MXOnly-1U-Hotswap-180")
     )
     (path "/00000000-0000-0000-0000-000061dc7e3e"
-      (reference "SW_5_10") (unit 1) (value "MX-compatible or Kailh Choc v1") (footprint "ProjectLocal:SW_MX_PG1350_NoLed")
+      (reference "SW_5_10") (unit 1) (value "MX-compatible or Kailh Choc v1") (footprint "ProjectLocal:MXOnly-1U-Hotswap-180")
     )
     (path "/00000000-0000-0000-0000-000061dc833b"
-      (reference "SW_5_11") (unit 1) (value "MX-compatible or Kailh Choc v1") (footprint "ProjectLocal:SW_MX_PG1350_NoLed")
+      (reference "SW_5_11") (unit 1) (value "MX-compatible or Kailh Choc v1") (footprint "ProjectLocal:MXOnly-1U-Hotswap-180")
     )
     (path "/00000000-0000-0000-0000-000061dc86c0"
-      (reference "SW_5_12") (unit 1) (value "MX-compatible or Kailh Choc v1") (footprint "ProjectLocal:SW_MX_PG1350_NoLed")
+      (reference "SW_5_12") (unit 1) (value "MX-compatible or Kailh Choc v1") (footprint "ProjectLocal:MXOnly-1U-Hotswap-180")
     )
     (path "/00000000-0000-0000-0000-000061af765f"

Commit message: fix: change switch symbol value to mx hotswap
Parts:
- SW_1_1, SW_1_10, SW_1_11, SW_1_12, SW_1_2, SW_1_3, SW_1_4, SW_1_5, SW_1_6, SW_1_7, SW_1_8, SW_1_9, SW_2_1, SW_2_10, SW_2_11, SW_2_12, SW_2_2, SW_2_3, SW_2_4, SW_2_5, SW_2_6, SW_2_7, SW_2_8, SW_2_9, SW_3_1, SW_3_10, SW_3_11, SW_3_12, SW_3_2, SW_3_3, SW_3_4, SW_3_5, SW_3_6, SW_3_7, SW_3_8, SW_3_9, SW_4_1, SW_4_10, SW_4_11, SW_4_12, SW_4_2, SW_4_3, SW_4_4, SW_4_5, SW_4_6, SW_4_7, SW_4_8, SW_4_9, SW_5_1, SW_5_10, SW_5_11, SW_5_12, SW_5_2, SW_5_3, SW_5_4, SW_5_5, SW_5_6, SW_5_7, SW_5_8, SW_5_9: value MX-compatible or Kailh Choc v1 -> MX Hotswap
